File: hw/tx-1/qse-mux.kicad_sch (KiCad schematic)
At the start: 4 parts, among them U3 SN74CBT3253

Commit message: Working on TX
Parts:
- added C23: 4.7uF, Capacitor_SMD:C_0805_2012Metric_Pad1.18x1.45mm_HandSolder, symbol Device:C_Small
- added R13: 2.2k, Resistor_SMD:R_0805_2012Metric_Pad1.20x1.40mm_HandSolder, symbol Device:R_Small_US
- added R14: 3.3k, Resistor_SMD:R_0805_2012Metric_Pad1.20x1.40mm_HandSolder, symbol Device:R_Small_US
- added R15, R16: 50, Resistor_SMD:R_0805_2012Metric_Pad1.20x1.40mm_HandSolder, symbol Device:R_Small_US
- C21, C22: footprint (none) -> Capacitor_SMD:C_0805_2012Metric_Pad1.18x1.45mm_HandSolder
- U3: footprint (none) -> Package_SO:SOIC-16_3.9x9.9mm_P1.27mm
Connections:
- net +5V: now also R14.1
- net GND: now also C22.2, TR1.4, C23.2, R13.2
- net at U3.7 (1A): now also R15.1; no longer TR1.5
- net at U3.9 (2A): now also R16.1; no longer TR1.8
- net at C22.1: now also TR1.6, TR1.7, C23.1, R13.1, R14.2
- net TX_OUT: now reaches TR1.1
- new net: R16.2, TR1.8
- new net: R15.2, TR1.5
Other:
- company: (none) -> KC1FSZ - Bruce MacKinnon 
- title: (none) -> Quadrature Transmit Board
- moved on the sheet: C22
