File: hw/tx-1/qse.kicad_sch (KiCad schematic)
At the start: 34 parts, among them U1 LM4562, U2 LM4562

Commit message: Working on TX
Parts:
- added C24: 4.7uF, Capacitor_SMD:C_0805_2012Metric_Pad1.18x1.45mm_HandSolder, symbol Device:C_Small
- added C25: 0.1uF, Capacitor_SMD:C_0805_2012Metric_Pad1.18x1.45mm_HandSolder, symbol Device:C_Small
- added R17, R18: 2.2k, Resistor_SMD:R_0805_2012Metric_Pad1.20x1.40mm_HandSolder, symbol Device:R_Small_US
- C1, C10, C11, C12, C13, C14, C15, C16, C17, C18, C19, C2, C20, C3, C4, C5, C6, C7, C8, C9: footprint (none) -> Capacitor_SMD:C_0805_2012Metric_Pad1.18x1.45mm_HandSolder
- R1, R10, R11, R12, R2, R3, R4, R5, R6, R7, R8, R9: footprint (none) -> Resistor_SMD:R_0805_2012Metric_Pad1.20x1.40mm_HandSolder
- U1, U2: footprint (none) -> Package_SO:SOIC-8_3.9x4.9mm_P1.27mm
Connections:
- net +5V: now also R17.1
- net GND: now also C24.2, C25.2, R18.2
- net VBIAS: now also C24.1, C25.1, R17.2, R18.1
- net I_OUT renamed I_IN
- net Q_OUT renamed Q_IN
Other:
- note added: "2.5V Bias Voltage"
- company: (none) -> KC1FSZ - Bruce MacKinnon 
- title: (none) -> Quadrature Transmit Board
