File: hw/tx-1/tx-1.kicad_sch (KiCad schematic)
At the start: 0 parts

Commit message: Working on TX
Parts:
- added H1, H2, H3, H4: MountingHole, MountingHole:MountingHole_3.5mm, symbol Mechanical:MountingHole
- added J1, J3: Conn_01x04, Connector_PinHeader_2.54mm:PinHeader_1x04_P2.54mm_Vertical, symbol Connector_Generic:Conn_01x04
- added J2, J4: Conn_01x02, Connector_PinHeader_2.54mm:PinHeader_1x02_P2.54mm_Vertical, symbol Connector_Generic:Conn_01x02
Connections:
- new net +5V: J2.1 (Pin_1)
- new net CLK_I: J3.1 (Pin_1)
- new net CLK_Q: J3.3 (Pin_3)
- new net GND: J1.2 (Pin_2), J1.4 (Pin_4), J2.2 (Pin_2), J3.2 (Pin_2), J3.4 (Pin_4), J4.2 (Pin_2)
- new net I_IN: J1.1 (Pin_1)
- new net Q_IN: J1.3 (Pin_3)
- new net TX_OUT: J4.1 (Pin_1)
Other:
- company: (none) -> KC1FSZ - Bruce MacKinnon 
- title: (none) -> Quadrature Transmit Board
