File: hw/tx-1/tx-1.kicad_pcb (KiCad board)
At the start: 2 copper layers, 68 x 41 mm, 55 parts, among them J1 Conn_01x04, J2 Conn_01x02, J3 Conn_01x04, J4 Conn_01x02, U1 LM4562, U2 LM4562, U3 SN74CBT3253

Commit message: Ready to sent to fab
Routing:
- net CLK_Q: track 13.6 -> 11.9 mm
Other:
- board text added: "5V"
- board text added: "GND"
- board text added: "OUT"
Changed lines of the file:
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@@
 			(plot_on_all_layers_selection 0x0000000_00000000)
 			(disableapertmacros no)
-			(usegerberextensions no)
-			(usegerberattributes yes)
-			(usegerberadvancedattributes yes)
-			(creategerberjobfile yes)
+			(usegerberextensions yes)
+			(usegerberattributes no)
+			(usegerberadvancedattributes no)
+			(creategerberjobfile no)
 			(dashed_line_dash_ratio 12.000000)
 			(dashed_line_gap_ratio 3.000000)
@@
 			(psa4output no)
 			(plotreference yes)
-			(plotvalue yes)
+			(plotvalue no)
 			(plotfptext yes)
 			(plotinvisibletext no)
 			(sketchpadsonfab no)
-			(subtractmaskfromsilk no)
+			(subtractmaskfromsilk yes)
 			(outputformat 1)
 			(mirror no)
-			(drillshape 1)
+			(drillshape 0)
 			(scaleselection 1)
-			(outputdirectory "")
+			(outputdirectory "plots")
 		)
 	)
@@
 		(tags "resistor handsolder")
 		(property "Reference" "R18"
-			(at 0 -1.65 360)
+			(at 0 -2 360)
 			(layer "F.SilkS")
 			(effects
@@
 		(layer "Edge.Cuts")
 	)
+	(gr_text "OUT"
+		(at 186 91.5 0)
+		(layer "F.SilkS")
+		(effects
+			(font
+				(size 0.8 0.8)
+				(thickness 0.1)
+			)
+			(justify left bottom)
+		)
+	)
 	(gr_text "KC1FSZ - 2025-01"
 		(at 134 103 0)
@@
 		)
 	)
+	(gr_text "5V"
+		(at 127.5 71.5 0)
+		(layer "F.SilkS")
+		(effects
+			(font
+				(size 0.8 0.8)
+				(thickness 0.09375)
+			)
+			(justify left bottom)
+		)
+	)
+	(gr_text "GND"
+		(at 126.5 74 0)
+		(layer "F.SilkS")
+		(effects
+			(font
+				(size 0.8 0.8)
+				(thickness 0.09375)
+			)
+			(justify left bottom)
+		)
+	)
 	(segment
 		(start 127.925 81.075)
@@
 	)
 	(segment
-		(start 169.974999 79.825)
-		(end 171.61 78.189999)
-		(width 0.2)
-		(layer "F.Cu")
-		(net 24)
-	)
-	(segment
-		(start 169.5 73)
-		(end 170.22 72.28)
+		(start 170.275 69.055)
+		(end 170.275 79.524999)
 		(width 0.2)
 		(layer "F.Cu")
@@
 	)
 	(segment
-		(start 169 79.825)
+		(start 170.275 79.524999)
 		(end 169.974999 79.825)
 		(width 0.2)
@@
 	)
 	(segment
-		(start 171.61 76.11)
-		(end 169.5 74)
+		(start 170.22 69)
+		(end 170.275 69.055)
 		(width 0.2)
 		(layer "F.Cu")
@@
 	)
 	(segment
-		(start 169.5 74)
-		(end 169.5 73)
-		(width 0.2)
-		(layer "F.Cu")
-		(net 24)
-	)
-	(segment
-		(start 170.22 72.28)
-		(end 170.22 69)
-		(width 0.2)
-		(layer "F.Cu")
-		(net 24)
-	)
-	(segment
-		(start 171.61 78.189999)
-		(end 171.61 76.11)
+		(start 169.974999 79.825)
+		(end 169 79.825)
 		(width 0.2)
 		(layer "F.Cu")
