File: hw/audio-breakout/adc.kicad_sch (KiCad schematic)
At the start: 18 parts, among them U2 PCM1804DBR

Commit message: New board for power, etc
Connections:
- net GND: no longer U2.12 (BYPAS)
- new net HPFBYPASS: U2.12 (BYPAS)
Changed lines of the file:
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@@
 	(title_block
 		(title "Digital Audio Breakout Board")
-		(date "2025-01-26")
-		(rev "1")
+		(date "2025-02-05")
+		(rev "2")
 		(company "Bruce MacKinnon KC1FSZ")
 		(comment 1 "Copyright (C) 2025")
@@
 	)
 	(junction
-		(at 91.44 116.84)
-		(diameter 0)
-		(color 0 0 0 0)
-	)
-	(junction
 		(at 231.14 88.9)
 		(diameter 0)
@@
 	(wire
 		(pts
-			(xy 91.44 91.44) (xy 91.44 116.84)
+			(xy 91.44 91.44) (xy 91.44 119.38)
 		)
 		(stroke
@@
 	(wire
 		(pts
-			(xy 91.44 116.84) (xy 100.33 116.84)
-		)
-		(stroke
-			(width 0)
-			(type default)
-		)
-	)
-	(wire
-		(pts
 			(xy 185.42 91.44) (xy 185.42 101.6)
 		)
@@
 	(wire
 		(pts
-			(xy 91.44 116.84) (xy 91.44 119.38)
-		)
-		(stroke
-			(width 0)
-			(type default)
-		)
-	)
-	(wire
-		(pts
 			(xy 251.46 105.41) (xy 251.46 104.14)
 		)
@@
 		(pts
 			(xy 67.31 106.68) (xy 100.33 106.68)
+		)
+		(stroke
+			(width 0)
+			(type default)
+		)
+	)
+	(wire
+		(pts
+			(xy 60.96 116.84) (xy 100.33 116.84)
 		)
 		(stroke
@@
 				(hide yes)
 			)
+		)
+	)
+	(global_label "HPFBYPASS"
+		(shape input)
+		(at 60.96 116.84 180)
+		(fields_autoplaced yes)
+		(effects
+			(font
+				(size 1.27 1.27)
+			)
+			(justify right)
+		)
+		(property "Intersheetrefs" "${INTERSHEET_REFS}"
+			(at 47.1495 116.84 0)
+			(effects
+				(font
+					(size 1.27 1.27)
+				)
+				(justify right)
+				(hide yes)
+			)
