File: hw/audio-breakout/audio-breakout.kicad_pcb (KiCad board)
At the start: 2 copper layers, 76.2 x 41.5 mm, 46 parts, among them J1 Conn_01x03, J2 Conn_01x04, J3 Conn_01x05, J4 Conn_01x04, J5 Conn_01x04, U1 PCM5100, U2 PCM1804DBR

Commit message: New board for power, etc
Other:
- board text added: "KC1FSZ - 2025-02"
- board text removed: "KC1FSZ - 2025-01"
Changed lines of the file:
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@@
 		(tags "resistor handsolder")
 		(property "Reference" "R1"
-			(at -3 0 360)
+			(at -3 0 0)
 			(layer "F.SilkS")
 			(effects
@@
 		)
 		(property "Value" "470"
-			(at 0 1.65 360)
+			(at 0 1.65 0)
 			(layer "F.Fab")
 			(effects
@@
 		)
 		(fp_text user "${REFERENCE}"
-			(at 0 0 360)
+			(at 0 0 0)
 			(layer "F.Fab")
 			(effects
@@
 		)
 		(fp_text user "${REFERENCE}"
-			(at 0 5.08 360)
+			(at 0 5.08 0)
 			(layer "F.Fab")
 			(effects
@@
 		(tags "net tie solder jumper bridged")
 		(property "Reference" "JP2"
-			(at 3.7 -0.45 360)
+			(at 3.7 -0.45 0)
 			(layer "F.SilkS")
 			(effects
@@
 		)
 		(property "Value" "SolderJumper_3_Bridged12"
-			(at 0 2 360)
+			(at 0 2 0)
 			(layer "F.Fab")
 			(effects
@@
 		(tags "net tie solder jumper bridged")
 		(property "Reference" "JP8"
-			(at 4.2 0 360)
+			(at 4.2 0 0)
 			(layer "F.SilkS")
 			(effects
@@
 		)
 		(property "Value" "SolderJumper_3_Bridged12"
-			(at 0 2 360)
+			(at 0 2 0)
 			(layer "F.Fab")
 			(effects
@@
 		(tags "capacitor handsolder")
 		(property "Reference" "C7"
-			(at 3.5 0 360)
+			(at 3.5 0 0)
 			(layer "F.SilkS")
 			(effects
@@
 		)
 		(property "Value" "0.1uF"
-			(at 0 1.68 360)
+			(at 0 1.68 0)
 			(layer "F.Fab")
 			(effects
@@
 		)
 		(fp_text user "${REFERENCE}"
-			(at 0 0 360)
+			(at 0 0 0)
 			(layer "F.Fab")
 			(effects
@@
 		(tags "TSSOP SO")
 		(property "Reference" "U1"
-			(at 0 -4.2 360)
+			(at 0 -4.2 0)
 			(layer "F.SilkS")
 			(effects
@@
 		)
 		(property "Value" "PCM5100"
-			(at 0 4.2 360)
+			(at 0 4.2 0)
 			(layer "F.Fab")
 			(effects
@@
 		)
 		(property "Footprint" "Package_SO:TSSOP-20_4.4x6.5mm_P0.65mm"
-			(at 0 0 360)
+			(at 0 0 0)
 			(layer "F.Fab")
 			(hide yes)
@@
 		)
 		(property "Datasheet" "http://www.ti.com/lit/ds/symlink/pcm5100.pdf"
-			(at 0 0 360)
+			(at 0 0 0)
 			(layer "F.Fab")
 			(hide yes)
@@
 		)
 		(property "Description" "2VRMS DirectPath, 100dB Audio Stereo DAC with 32-bit, 384kHz PCM Interface, TSSOP-20"
-			(at 0 0 360)
+			(at 0 0 0)
 			(layer "F.Fab")
 			(hide yes)
@@
 		)
 		(fp_text user "${REFERENCE}"
-			(at 0 0 360)
+			(at 0 0 0)
 			(layer "F.Fab")
 			(effects
@@
 		(tags "net tie solder jumper bridged")
 		(property "Reference" "JP4"
-			(at -3.7 0.6 360)
+			(at -3.7 0.6 0)
 			(layer "F.SilkS")
 			(effects
@@
 		)
 		(property "Value" "SolderJumper_3_Bridged12"
-			(at 0 2 360)
+			(at 0 2 0)
 			(layer "F.Fab")
 			(effects
@@
 		(tags "net tie solder jumper bridged")
 		(property "Reference" "JP13"
-			(at 4.5 0 360)
+			(at 4.5 0 0)
 			(layer "F.SilkS")
 			(effects
@@
 		)
 		(property "Value" "SolderJumper_3_Bridged12"
-			(at 0 2 360)
+			(at 0 2 0)
 			(layer "F.Fab")
 			(effects
@@
 		(tags "capacitor handsolder")
 		(property "Reference" "C12"
-			(at 4 0 360)
+			(at 4 0 0)
 			(layer "F.SilkS")
 			(effects
@@
 		)
 		(property "Value" "1u"
-			(at 0 1.68 360)
+			(at 0 1.68 0)
 			(layer "F.Fab")
 			(effects
@@
 		)
 		(fp_text user "${REFERENCE}"
-			(at 0 0 360)
+			(at 0 0 0)
 			(layer "F.Fab")
 			(effects
@@
 		)
 		(fp_text user "${REFERENCE}"
-			(at 0 3.81 360)
+			(at 0 3.81 0)
 			(layer "F.Fab")
 			(effects
@@
 		(tags "net tie solder jumper bridged")
 		(property "Reference" "JP9"
-			(at -4 0 360)
+			(at -4 0 0)
 			(layer "F.SilkS")
 			(effects
@@
 		)
 		(property "Value" "SolderJumper_3_Bridged12"
-			(at 0 2 360)
+			(at 0 2 0)
 			(layer "F.Fab")
 			(effects
@@
 		(tags "Through hole pin header THT 1x04 2.54mm single row")
 		(property "Reference" "J5"
-			(at 0 -2.33 360)
+			(at 0 -2.33 0)
 			(layer "F.SilkS")
 			(effects
@@
 		)
 		(property "Value" "Conn_01x04"
-			(at 0 9.95 360)
+			(at 0 9.95 0)
 			(layer "F.Fab")
 			(effects
@@
 		(tags "net tie solder jumper bridged")
 		(property "Reference" "JP12"
-			(at -4.5 0 360)
+			(at -4.5 0 0)
 			(layer "F.SilkS")
 			(effects
@@
 		)
 		(property "Value" "SolderJumper_3_Bridged12"
-			(at 0 2 360)
+			(at 0 2 0)
 			(layer "F.Fab")
 			(effects
@@
 		(tags "capacitor handsolder")
 		(property "Reference" "C9"
-			(at -3 0 360)
+			(at -3 0 0)
 			(layer "F.SilkS")
 			(effects
@@
 		)
 		(property "Value" "2.2nF"
-			(at 0 1.68 360)
+			(at 0 1.68 0)
 			(layer "F.Fab")
 			(effects
@@
 		)
 		(fp_text user "${REFERENCE}"
-			(at 0 0 360)
+			(at 0 0 0)
 			(layer "F.Fab")
 			(effects
@@
 		(tags "capacitor handsolder")
 		(property "Reference" "C3"
-			(at -3 0 360)
+			(at -3 0 0)
 			(layer "F.SilkS")
 			(effects
@@
 		)
 		(property "Value" "2.2uF"
-			(at 0 1.68 360)
+			(at 0 1.68 0)
 			(layer "F.Fab")
 			(effects
@@
 		)
 		(fp_text user "${REFERENCE}"
-			(at 0 0 360)
+			(at 0 0 0)
 			(layer "F.Fab")
 			(effects
@@
 		(tags "resistor handsolder")
 		(property "Reference" "R2"
-			(at -3 0 360)
+			(at -3 0 0)
 			(layer "F.SilkS")
 			(effects
@@
 		)
 		(property "Value" "470"
-			(at 0 1.65 360)
+			(at 0 1.65 0)
 			(layer "F.Fab")
 			(effects
@@
 		)
 		(fp_text user "${REFERENCE}"
-			(at 0 0 360)
+			(at 0 0 0)
 			(layer "F.Fab")
 			(effects
@@
 		(tags "net tie solder jumper bridged")
 		(property "Reference" "JP11"
-			(at -4.5 0 360)
+			(at -4.5 0 0)
 			(layer "F.SilkS")
 			(effects
@@
 		)
 		(property "Value" "SolderJumper_3_Bridged12"
-			(at 0 2 360)
+			(at 0 2 0)
 			(layer "F.Fab")
 			(effects
@@
 		(tags "net tie solder jumper bridged")
 		(property "Reference" "JP10"
-			(at 4.45 0 360)
+			(at 4.45 0 0)
 			(layer "F.SilkS")
 			(effects
@@
 		)
 		(property "Value" "SolderJumper_3_Bridged12"
-			(at 0 2 360)
+			(at 0 2 0)
 			(layer "F.Fab")
 			(effects
@@
 		(tags "net tie solder jumper bridged")
 		(property "Reference" "JP3"
-			(at 0.2 2.25 360)
+			(at 0.2 2.25 0)
 			(layer "F.SilkS")
 			(effects
@@
 		)
 		(property "Value" "SolderJumper_3_Bridged12"
-			(at 0 2 360)
+			(at 0 2 0)
 			(layer "F.Fab")
 			(effects
@@
 		(tags "net tie solder jumper bridged")
 		(property "Reference" "JP1"
-			(at -3.5 0.55 360)
+			(at -3.5 0.55 0)
 			(layer "F.SilkS")
 			(effects
@@
 		)
 		(property "Value" "SolderJumper_3_Bridged12"
-			(at 0 2 360)
+			(at 0 2 0)
 			(layer "F.Fab")
 			(effects
@@
 		)
 		(fp_text user "${REFERENCE}"
-			(at 0 3.81 360)
+			(at 0 3.81 0)
 			(layer "F.Fab")
 			(effects
@@
 		(tags "capacitor handsolder")
 		(property "Reference" "C5"
-			(at 3 0 360)
+			(at 3 0 0)
 			(layer "F.SilkS")
 			(effects
@@
 		)
 		(property "Value" "2.2uF"
-			(at 0 1.68 360)
+			(at 0 1.68 0)
 			(layer "F.Fab")
 			(effects
@@
 		)
 		(fp_text user "${REFERENCE}"
-			(at 0 0 360)
+			(at 0 0 0)
 			(layer "F.Fab")
 			(effects
@@
 		(tags "capacitor handsolder")
 		(property "Reference" "C8"
-			(at -3 0 360)
+			(at -3 0 0)
 			(layer "F.SilkS")
 			(effects
@@
 		)
 		(property "Value" "2.2nF"
-			(at 0 1.68 360)
+			(at 0 1.68 0)
 			(layer "F.Fab")
 			(effects
@@
 		)
 		(fp_text user "${REFERENCE}"
-			(at 0 0 360)
+			(at 0 0 0)
 			(layer "F.Fab")
 			(effects
@@
 		(tags "inductor handsolder")
 		(property "Reference" "L1"
-			(at -3 0 360)
+			(at -3 0 0)
 			(layer "F.SilkS")
 			(effects
@@
 		)
 		(property "Value" "47u"
-			(at 0 1.65 360)
+			(at 0 1.65 0)
 			(layer "F.Fab")
 			(effects
@@
 		)
 		(fp_text user "${REFERENCE}"
-			(at 0 0 360)
+			(at 0 0 0)
 			(layer "F.Fab")
 			(effects
@@
 		)
 	)
-	(gr_text "KC1FSZ - 2025-01"
+	(gr_text "KC1FSZ - 2025-02"
 		(at 164 130.25 0)
 		(layer "F.SilkS")
