File: hw/audio-breakout/audio-breakout.kicad_sch (KiCad schematic)
At the start: 12 parts, among them J1 Conn_01x03, J2 Conn_01x04, J3 Conn_01x05, J4 Conn_01x04, J5 Conn_01x04

Commit message: New board for power, etc
Parts:
- added J6: Conn_01x02, symbol Connector_Generic:Conn_01x02
Connections:
- net GND: now also J6.2 (Pin_2)
- new net HPFBYPASS: J6.1 (Pin_1)
Other:
- note added: "Control for ADC high-pass filter bypass. Low=normal (i.e. not bypassed), High=bypassed. This is useful for enabling DC calibration of the ADC."
- note added: "Optional feature to allow the I2S clock lines for the ADC and DAC to be connected. This could reduce MPU pin count when common clocks are possible."
- moved on the sheet: JP5, JP6, JP7
