File: hw/util-1/audio-out.kicad_sch (KiCad schematic)
At the start: 0 parts

Commit message: Initial version of PCB layout
Parts:
- added C3: 0.39uF, Capacitor_SMD:C_0805_2012Metric_Pad1.18x1.45mm_HandSolder, symbol Device:C
- added C4: 1.0uF, Capacitor_SMD:C_0805_2012Metric_Pad1.18x1.45mm_HandSolder, symbol Device:C
- added C7: NC, Capacitor_SMD:C_0805_2012Metric_Pad1.18x1.45mm_HandSolder, symbol Device:C
- added C8: 0.1uF, Capacitor_SMD:C_0805_2012Metric_Pad1.18x1.45mm_HandSolder, symbol Device:C
- added J4: Conn_01x02, Connector_PinHeader_2.54mm:PinHeader_1x02_P2.54mm_Vertical, symbol Connector_Generic:Conn_01x02
- added J5: Conn_01x06, Connector_PinHeader_2.54mm:PinHeader_1x06_P2.54mm_Vertical, symbol Connector_Generic:Conn_01x06
- added R1, R3: 20k, Resistor_SMD:R_0805_2012Metric_Pad1.20x1.40mm_HandSolder, symbol Device:R
- added R4: 1k, Resistor_SMD:R_0805_2012Metric_Pad1.20x1.40mm_HandSolder, symbol Device:R_Small_US
- added U1: ~, Package_SO:SOIC-8_3.9x4.9mm_P1.27mm, symbol symbol-library-1:LM4862M
Connections:
- new net: C7.2, R1.2, R3.1, U1.4 (-IN)
- new net: C7.1, J4.2 (Pin_2), R3.2, U1.5 (Vo1)
- new net: C3.1, J5.2 (Pin_2)
- new net: C3.2, R1.1
- new net: J5.6 (Pin_6), R4.2, U1.1 (SHUTDOWN)
- new net: J5.3 (Pin_3), J5.4 (Pin_4)
- new net: C4.1, U1.2 (BYPASS), U1.3 (+IN)
- new net: J4.1 (Pin_1), U1.8 (Vo2)
- new net +5V: C8.1, R4.1, U1.6 (VDD)
- new net GND: C4.2, C8.2, J5.1 (Pin_1), J5.5 (Pin_5), U1.7 (GND)
Other:
- note added: "Optional, 22pF if used for stability."
- note added: "Speaker"
- company: (none) -> Bruce MacKinnon KC1FSZ
- title: (none) -> Utility Board 1
