File: hw/util-1/audio-in.kicad_sch (KiCad schematic)
At the start: 15 parts, among them J6 Conn_01x02, U4 MAX4466EXK

Commit message: Sending revision of util-1 to JLCPCB
Parts:
- removed FB2: FerriteBead, Inductor_SMD:L_0805_2012Metric_Pad1.15x1.40mm_HandSolder, symbol Device:FerriteBead
Connections:
- net GNDA is gone; now on net GND: C10.1, C11.1, J6.2 (Pin_2), R8.2, U4.2 (GND)
