File: hw/txrx-1/qse-mux.kicad_sch (KiCad schematic)
At the start: 9 parts, among them U43 SN74CBT3253

Commit message: Initial PCB layout for TXRX board
Other:
- company: (none) -> Bruce MacKinnon KC1FSZ
- title: (none) -> Quadrature TX/RX Board
Changed lines of the file:
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@@
 	(generator "eeschema")
 	(generator_version "8.0")
-	(paper "A4")
+	(paper "USLetter")
+	(title_block
+		(title "Quadrature TX/RX Board")
+		(date "2025-02-16")
+		(rev "1")
+		(company "Bruce MacKinnon KC1FSZ")
+		(comment 1 "Copyright (C) Bruce MacKinnon, 2025")
+		(comment 2 "NOT FOR COMMERCIAL USE")
+	)
 	(junction
 		(at 95.25 90.17)

Commit message: Final version being sent to fab
Parts:
- added R70, R71: 0, Resistor_SMD:R_0805_2012Metric_Pad1.20x1.40mm_HandSolder, symbol Device:R_Small_US
- C64: value 4.7uF -> 10uF
Connections:
- net CLK_I: now also R70.2; no longer U43.14 (S0)
- net CLK_Q: now also R71.2; no longer U43.2 (S1)
- new net: R70.1, U43.14 (S0)
- new net: R71.1, U43.2 (S1)
Other:
- note added: "0ohm for cross-over on PCB"
Changed lines of the file:
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@@
 	(title_block
 		(title "Quadrature TX/RX Board")
-		(date "2025-02-16")
+		(date "2025-02-17")
 		(rev "1")
 		(company "Bruce MacKinnon KC1FSZ")
@@
 	(wire
 		(pts
+			(xy 132.08 100.33) (xy 142.24 100.33)
+		)
+		(stroke
+			(width 0)
+			(type default)
+		)
+	)
+	(wire
+		(pts
 			(xy 82.55 92.71) (xy 93.98 92.71)
 		)
@@
 	(wire
 		(pts
-			(xy 132.08 97.79) (xy 147.32 97.79)
-		)
-		(stroke
-			(width 0)
-			(type default)
-		)
-	)
-	(wire
-		(pts
 			(xy 147.32 87.63) (xy 195.58 87.63)
 		)
@@
 	(wire
 		(pts
+			(xy 147.32 100.33) (xy 160.02 100.33)
+		)
+		(stroke
+			(width 0)
+			(type default)
+		)
+	)
+	(wire
+		(pts
 			(xy 205.74 90.17) (xy 217.17 90.17)
 		)
@@
 	(wire
 		(pts
-			(xy 132.08 100.33) (xy 160.02 100.33)
-		)
-		(stroke
-			(width 0)
-			(type default)
-		)
-	)
-	(wire
-		(pts
 			(xy 121.92 71.12) (xy 102.87 71.12)
 		)
@@
 	(wire
 		(pts
+			(xy 142.24 97.79) (xy 147.32 97.79)
+		)
+		(stroke
+			(width 0)
+			(type default)
+		)
+	)
+	(wire
+		(pts
 			(xy 191.77 95.25) (xy 195.58 95.25)
 		)
@@
 	(wire
 		(pts
+			(xy 132.08 97.79) (xy 137.16 97.79)
+		)
+		(stroke
+			(width 0)
+			(type default)
+		)
+	)
+	(wire
+		(pts
 			(xy 191.77 109.22) (xy 191.77 113.03)
 		)
@@
 			(width 0)
 			(type default)
+		)
+	)
+	(text "0ohm for cross-over on PCB"
+		(exclude_from_sim no)
+		(at 148.082 103.124 0)
+		(effects
+			(font
+				(size 1.27 1.27)
+			)
 		)
 	)
@@
 	)
 	(symbol
+		(lib_id "Device:R_Small_US")
+		(at 139.7 97.79 90)
+		(unit 1)
+		(exclude_from_sim no)
+		(in_bom yes)
+		(on_board yes)
+		(dnp no)
+		(property "Reference" "R70"
+			(at 139.7 92.71 90)
+			(effects
+				(font
+					(size 1.27 1.27)
+				)
+			)
+		)
+		(property "Value" "0"
+			(at 139.7 95.25 90)
+			(effects
+				(font
+					(size 1.27 1.27)
+				)
+			)
+		)
+		(property "Footprint" "Resistor_SMD:R_0805_2012Metric_Pad1.20x1.40mm_HandSolder"
+			(at 139.7 97.79 0)
+			(effects
+				(font
+					(size 1.27 1.27)
+				)
+				(hide yes)
+			)
+		)
+		(property "Datasheet" "~"
+			(at 139.7 97.79 0)
+			(effects
+				(font
+					(size 1.27 1.27)
+				)
+				(hide yes)
+			)
+		)
+		(property "Description" "Resistor, small US symbol"
+			(at 139.7 97.79 0)
+			(effects
+				(font
+					(size 1.27 1.27)
+				)
+				(hide yes)
+			)
+		)
+		(pin "1"
+		)
+		(pin "2"
+		)
+		(instances
+			(project "txrx-1"
+				(path "/8e82f983-38e6-4304-be32-fb6d88cc8acc/7ed2824d-e7e3-4e73-ad8c-26a3a131b178/a50ce90c-3197-46da-9f0b-d409feefa4c7"
+					(reference "R70")
+					(unit 1)
+				)
+			)
+		)
+	)
+	(symbol
 		(lib_id "power:GND")
 		(at 176.53 118.11 0)
@@
 	)
 	(symbol
+		(lib_id "Device:R_Small_US")
+		(at 144.78 100.33 90)
+		(unit 1)
+		(exclude_from_sim no)
+		(in_bom yes)
+		(on_board yes)
+		(dnp no)
+		(property "Reference" "R71"
+			(at 144.78 95.25 90)
+			(effects
+				(font
+					(size 1.27 1.27)
+				)
+			)
+		)
+		(property "Value" "0"
+			(at 144.78 97.79 90)
+			(effects
+				(font
+					(size 1.27 1.27)
+				)
+			)
+		)
+		(property "Footprint" "Resistor_SMD:R_0805_2012Metric_Pad1.20x1.40mm_HandSolder"
+			(at 144.78 100.33 0)
+			(effects
+				(font
+					(size 1.27 1.27)
+				)
+				(hide yes)
+			)
+		)
+		(property "Datasheet" "~"
+			(at 144.78 100.33 0)
+			(effects
+				(font
+					(size 1.27 1.27)
+				)
+				(hide yes)
+			)
+		)
+		(property "Description" "Resistor, small US symbol"
+			(at 144.78 100.33 0)
+			(effects
+				(font
+					(size 1.27 1.27)
+				)
+				(hide yes)
+			)
+		)
+		(pin "1"
+		)
+		(pin "2"
+		)
+		(instances
+			(project "txrx-1"
+				(path "/8e82f983-38e6-4304-be32-fb6d88cc8acc/7ed2824d-e7e3-4e73-ad8c-26a3a131b178/a50ce90c-3197-46da-9f0b-d409feefa4c7"
+					(reference "R71")
+					(unit 1)
+				)
+			)
+		)
+	)
+	(symbol
 		(lib_id "power:+5V")
 		(at 191.77 73.66 0)
@@
 			)
 		)
-		(property "Value" "4.7uF"
+		(property "Value" "10uF"
 			(at 166.37 116.8462 0)
 			(effects
