File: hw/txrx-1/tx.kicad_sch (KiCad schematic)
At the start: 0 parts

Commit message: Initial PCB layout for TXRX board
Other:
- company: (none) -> Bruce MacKinnon KC1FSZ
- title: (none) -> Quadrature TX/RX Board
Changed lines of the file:
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@@
 	(generator "eeschema")
 	(generator_version "8.0")
-	(paper "A4")
+	(paper "USLetter")
+	(title_block
+		(title "Quadrature TX/RX Board")
+		(date "2025-02-16")
+		(rev "1")
+		(company "Bruce MacKinnon KC1FSZ")
+		(comment 1 "Copyright (C) Bruce MacKinnon, 2025")
+		(comment 2 "NOT FOR COMMERCIAL USE")
+	)
 	(sheet
 		(at 76.2 24.13)
