File: hw/bpf-1/bpf-1.kicad_pcb (KiCad board)
At the start: 2 copper layers, 25 x 70 mm, 31 parts, among them J1 Conn_01x04, J2 Conn_01x02, J3 Conn_01x02, U1 SN74CBT3253

Commit message: Ready to send to fab
Parts:
- moved J3 2.50 mm to (184.0, 55.0), turned to 0 degrees
- moved J2 0.23 mm to (166.0, 55.0)
Routing:
- net BPF_O: track 15.2 -> 16.5 mm
- net BPF_I: track 6.75 -> 7.62 mm
- net GND: vias 17 -> 18
Other:
- board text added: "5V"
- board text added: "G"
- board text added: "IN"
- board text added: "OUT"
- board text added: "S0"
- board text added: "S1"
